Commit message: latest_navigation

File: src/app_robot_state_publisher/config/URDF/robot.urdf (robot description, URDF)
Before this commit: robot morpheus_rover, 29 links, 28 joints
Links:
- added link os_sensor
- added link zed_camera_link
Joints:
- added joint os_sensor_bridge_joint: type fixed, parent os0_lidar_link, child os_sensor
- added joint zed_camera_bridge_joint: type fixed, parent zed_2i_link, child zed_camera_link

Commit message: urdf fixes, rtabmap fixes

File: src/app_robot_state_publisher/config/URDF/robot.urdf (robot description, URDF)
Before this commit: robot morpheus_rover, 31 links, 30 joints
Joints:
- joint os0_lidar_joint: origin xyz=0.0 0.0 1.0 rpy=0.0 0.0 0.0 -> xyz=0.285 -0.155 0.17 rpy=0.0 0.0 0.0
- joint zed_2i_joint: origin xyz=0.35 0.0 0.0 rpy=0.0 0.0 0.0 -> xyz=0.35 0.0 0.106 rpy=0.0 0.0 0.0

Commit message: urdf naming convention correction

File: src/app_robot_state_publisher/config/URDF/robot.urdf (robot description, URDF)
Before this commit: robot morpheus_rover, 31 links, 30 joints
Links:
- removed link zed_camera_link
- added link zed2i_camera_link
Joints:
- joint zed_camera_bridge_joint: child zed_camera_link -> zed2i_camera_link

Commit message: Update configs, docker setup, and diagnostics

File: src/app_robot_state_publisher/config/URDF/robot.urdf (robot description, URDF)
Before this commit: robot morpheus_rover, 31 links, 30 joints
Links:
- added link zed2i_camera_center
- added link zed2i_left_camera_frame
- added link zed2i_left_camera_frame_optical
- added link zed2i_right_camera_frame
- added link zed2i_right_camera_frame_optical
Joints:
- added joint zed2i_camera_center_joint: type fixed, parent zed2i_camera_link, child zed2i_camera_center, origin xyz=0 0 0.015 rpy=0 0 0
- added joint zed2i_left_camera_joint: type fixed, parent zed2i_camera_center, child zed2i_left_camera_frame, origin xyz=-0.01 0.06 0 rpy=0 0 0
- added joint zed2i_left_camera_optical_joint: type fixed, parent zed2i_left_camera_frame, child zed2i_left_camera_frame_optical, origin xyz=0 0 0 rpy=-1.5708 0 -1.5708
- added joint zed2i_right_camera_joint: type fixed, parent zed2i_camera_center, child zed2i_right_camera_frame, origin xyz=-0.01 -0.06 0 rpy=0 0 0
- added joint zed2i_right_camera_optical_joint: type fixed, parent zed2i_right_camera_frame, child zed2i_right_camera_frame_optical, origin xyz=0 0 0 rpy=-1.5708 0 -1.5708

Commit message: moved lnew imu link to urdf

File: src/app_robot_state_publisher/config/URDF/robot.urdf (robot description, URDF)
Before this commit: robot morpheus_rover, 36 links, 35 joints
Links:
- added link imu_link
Joints:
- added joint imu_link_joint: type fixed, parent chassis_link, child imu_link, origin xyz=0.15 0.0 0.10 rpy=0 0 0
